File: Schematische tekeningen/Totaalschema/Voeding.sch (KiCad schematic (older format))
At the start: 19 parts

Commit message: Footprints toegevoegd en toegewezen. Tekening weer iets aangepast
Parts:
- C9: renamed from C?; footprint (none) -> Capacitor_SMD:C_0603_1608Metric_Pad1.08x0.95mm_HandSolder
- D2, D5: renamed from D?; footprint (none) -> Diode_SMD:D_SMC_Handsoldering
- D3: renamed from D?; footprint (none) -> Diode_SMD:D_SOD-323_HandSoldering
- D4: renamed from D?; footprint (none) -> Diode_SMD:D_PowerDI-123
- L1: renamed from L?; footprint (none) -> Inductor_SMD:L_10.4x10.4_H4.8
- R19, R20, R21, R22, R23, R24, R25: renamed from R?; footprint (none) -> Resistor_SMD:R_0603_1608Metric_Pad0.98x0.95mm_HandSolder
- T1: renamed from T?; footprint (none) -> eec:750313973
- U8: renamed from U?; footprint Linear_Technology-LT8301IS5TRPBF-* -> eec:Linear_Technology-LT8301IS5TRPBF-Level_A
- gave numbers to parts that had none: 4
Changed lines of the file:
@@
 $EndDescr
 $Comp
-L eec:LT8301IS5TRPBF U?
+L eec:LT8301IS5TRPBF U8
 U 1 1 6186DB9F
 P 3925 2600
-F 0 "U?" H 4525 2865 50  0000 C CNN
+F 0 "U8" H 4525 2865 50  0000 C CNN
 F 1 "LT8301IS5TRPBF" H 4525 2774 39  0000 C CNN
-F 2 "Linear_Technology-LT8301IS5TRPBF-*" H 3925 3000 50  0001 L CNN
+F 2 "eec:Linear_Technology-LT8301IS5TRPBF-Level_A" H 3925 3000 50  0001 L CNN
 F 3 "http://cds.linear.com/docs/en/datasheet/8301f.pdf" H 3925 3100 50  0001 L CNN
 F 4 "Manufacturer URL" H 3925 3200 50  0001 L CNN "Component Link 1 Description"
@@
 	5475 2600 5450 2600
 $Comp
-L Device:R_Small R?
+L Device:R_Small R22
 U 1 1 6186DBA7
 P 5475 2700
-F 0 "R?" H 5534 2746 50  0000 L CNN
+F 0 "R22" H 5534 2746 50  0000 L CNN
 F 1 "143k" H 5534 2655 39  0000 L CNN
-F 2 "" H 5475 2700 50  0001 C CNN
+F 2 "Resistor_SMD:R_0603_1608Metric_Pad0.98x0.95mm_HandSolder" H 5475 2700 50  0001 C CNN
 F 3 "~" H 5475 2700 50  0001 C CNN
 	1    5475 2700
@@
 $EndComp
 $Comp
-L Device:D_Schottky_Small D?
+L Device:D_Schottky_Small D5
 U 1 1 6186DBC1
 P 6350 2000
-F 0 "D?" H 6350 2100 50  0000 C CNN
+F 0 "D5" H 6350 2100 50  0000 C CNN
 F 1 "SS510" H 6350 1884 39  0000 C CNN
-F 2 "" V 6350 2000 50  0001 C CNN
+F 2 "Diode_SMD:D_SMC_Handsoldering" V 6350 2000 50  0001 C CNN
 F 3 "~" V 6350 2000 50  0001 C CNN
 	1    6350 2000
@@
 $EndComp
 $Comp
-L Device:C C?
+L Device:C C12
 U 1 1 6186DBC7
 P 6550 2150
-F 0 "C?" H 6665 2196 50  0000 L CNN
+F 0 "C12" H 6665 2196 50  0000 L CNN
 F 1 "85uF" H 6665 2105 39  0000 L CNN
 F 2 "" H 6588 2000 50  0001 C CNN
@@
 $EndComp
 $Comp
-L Device:R R?
+L Device:R R25
 U 1 1 6186DBCE
 P 6950 2150
-F 0 "R?" H 7020 2196 50  0000 L CNN
+F 0 "R25" H 7020 2196 50  0000 L CNN
 F 1 "390" H 7020 2105 50  0000 L CNN
-F 2 "" V 6880 2150 50  0001 C CNN
+F 2 "Resistor_SMD:R_0603_1608Metric_Pad0.98x0.95mm_HandSolder" V 6880 2150 50  0001 C CNN
 F 3 "~" H 6950 2150 50  0001 C CNN
 	1    6950 2150
@@
 $EndComp
 $Comp
-L power:GNDS #PWR?
+L power:GNDS #PWR039
 U 1 1 6186DBF0
 P 6950 2300
-F 0 "#PWR?" H 6950 2050 50  0001 C CNN
+F 0 "#PWR039" H 6950 2050 50  0001 C CNN
 F 1 "GNDS" H 6950 2150 50  0000 C CNN
 F 2 "" H 6950 2300 50  0001 C CNN
@@
 $EndComp
 $Comp
-L Device:C C?
+L Device:C C9
 U 1 1 6186DC04
 P 3625 2750
-F 0 "C?" H 3400 2775 50  0000 L CNN
+F 0 "C9" H 3400 2775 50  0000 L CNN
 F 1 "4,7u" H 3350 2700 39  0000 L CNN
-F 2 "" H 3663 2600 50  0001 C CNN
+F 2 "Capacitor_SMD:C_0603_1608Metric_Pad1.08x0.95mm_HandSolder" H 3663 2600 50  0001 C CNN
 F 3 "~" H 3625 2750 50  0001 C CNN
 	1    3625 2750
@@
 $EndComp
 $Comp
-L Device:R_Small R?
+L Device:R_Small R19
 U 1 1 6186DC0C
 P 3850 2700
-F 0 "R?" H 3909 2746 50  0000 L CNN
+F 0 "R19" H 3909 2746 50  0000 L CNN
 F 1 "232k" H 3909 2655 39  0000 L CNN
-F 2 "" H 3850 2700 50  0001 C CNN
+F 2 "Resistor_SMD:R_0603_1608Metric_Pad0.98x0.95mm_HandSolder" H 3850 2700 50  0001 C CNN
 F 3 "~" H 3850 2700 50  0001 C CNN
 	1    3850 2700
@@
 $EndComp
 $Comp
-L Device:R_Small R?
+L Device:R_Small R20
 U 1 1 6186DC14
 P 3850 2900
-F 0 "R?" H 3909 2946 50  0000 L CNN
+F 0 "R20" H 3909 2946 50  0000 L CNN
 F 1 "806k" H 3909 2855 39  0000 L CNN
-F 2 "" H 3850 2900 50  0001 C CNN
+F 2 "Resistor_SMD:R_0603_1608Metric_Pad0.98x0.95mm_HandSolder" H 3850 2900 50  0001 C CNN
 F 3 "~" H 3850 2900 50  0001 C CNN
 	1    3850 2900
@@
 VSS
 $Comp
-L Device:D_Zener_Small D?
+L Device:D_Zener_Small D3
 U 1 1 6186DB7B
 P 5450 2300
-F 0 "D?" V 5450 2500 50  0000 R CNN
+F 0 "D3" V 5450 2500 50  0000 R CNN
 F 1 "20V zener" V 5400 2650 39  0000 R CNN
-F 2 "" V 5450 2300 50  0001 C CNN
+F 2 "Diode_SMD:D_SOD-323_HandSoldering" V 5450 2300 50  0001 C CNN
 F 3 "~" V 5450 2300 50  0001 C CNN
 	1    5450 2300
@@
 $EndComp
 $Comp
-L Device:D_Schottky_Small D?
+L Device:D_Schottky_Small D4
 U 1 1 6186DB75
 P 5450 2500
-F 0 "D?" V 5350 2600 50  0000 L CNN
+F 0 "D4" V 5350 2600 50  0000 L CNN
 F 1 "1N4148" V 5450 2550 39  0000 L CNN
-F 2 "" V 5450 2500 50  0001 C CNN
+F 2 "Diode_SMD:D_PowerDI-123" V 5450 2500 50  0001 C CNN
 F 3 "~" V 5450 2500 50  0001 C CNN
 	1    5450 2500
@@
 	5450 2800 5475 2800
 $Comp
-L Device:R_Small R?
+L Device:R_Small R21
 U 1 1 619BE033
 P 5350 2800
-F 0 "R?" V 5275 2750 50  0000 L CNN
+F 0 "R21" V 5275 2750 50  0000 L CNN
 F 1 "1k" V 5350 2750 39  0000 L CNN
-F 2 "" H 5350 2800 50  0001 C CNN
+F 2 "Resistor_SMD:R_0603_1608Metric_Pad0.98x0.95mm_HandSolder" H 5350 2800 50  0001 C CNN
 F 3 "~" H 5350 2800 50  0001 C CNN
 	1    5350 2800
@@
 NoConn ~ 6250 2800
 $Comp
-L Regulator_Switching:LM2596S-ADJ U?
+L Regulator_Switching:LM2596S-ADJ U9
 U 1 1 61A475E3
 P 4575 3925
-F 0 "U?" H 4575 4292 50  0000 C CNN
+F 0 "U9" H 4575 4292 50  0000 C CNN
 F 1 "LM2596S-ADJ" H 4575 4201 50  0000 C CNN
 F 2 "Package_TO_SOT_SMD:TO-263-5_TabPin3" H 4625 3675 50  0001 L CIN
@@
 $EndComp
 $Comp
-L Device:C C?
+L Device:C C10
 U 1 1 61A48A94
 P 3725 3975
-F 0 "C?" H 3525 4025 50  0000 L CNN
+F 0 "C10" H 3525 4025 50  0000 L CNN
 F 1 "470u" H 3475 3900 50  0000 L CNN
 F 2 "" H 3763 3825 50  0001 C CNN
@@
 VSS
 $Comp
-L Device:L L?
+L Device:L L1
 U 1 1 61A51AA4
 P 5350 4025
-F 0 "L?" V 5540 4025 50  0000 C CNN
+F 0 "L1" V 5540 4025 50  0000 C CNN
 F 1 "68u" V 5449 4025 50  0000 C CNN
-F 2 "" H 5350 4025 50  0001 C CNN
+F 2 "Inductor_SMD:L_10.4x10.4_H4.8" H 5350 4025 50  0001 C CNN
 F 3 "~" H 5350 4025 50  0001 C CNN
 	1    5350 4025
@@
 $EndComp
 $Comp
-L Device:D_Schottky D?
+L Device:D_Schottky D2
 U 1 1 61A525B8
 P 5200 4175
-F 0 "D?" V 5154 4255 50  0000 L CNN
+F 0 "D2" V 5154 4255 50  0000 L CNN
 F 1 "SS310" V 5245 4255 50  0000 L CNN
-F 2 "" H 5200 4175 50  0001 C CNN
+F 2 "Diode_SMD:D_SMC_Handsoldering" H 5200 4175 50  0001 C CNN
 F 3 "~" H 5200 4175 50  0001 C CNN
 	1    5200 4175
@@
 Connection ~ 4575 4225
 $Comp
-L Device:C C?
+L Device:C C11
 U 1 1 61A760ED
 P 5600 4175
-F 0 "C?" H 5715 4221 50  0000 L CNN
+F 0 "C11" H 5715 4221 50  0000 L CNN
 F 1 "220u" H 5715 4130 50  0000 L CNN
 F 2 "" H 5638 4025 50  0001 C CNN
@@
 $EndComp
 $Comp
-L Device:R_Small R?
+L Device:R_Small R23
 U 1 1 61A8520F
 P 5975 4125
-F 0 "R?" H 6034 4171 50  0000 L CNN
+F 0 "R23" H 6034 4171 50  0000 L CNN
 F 1 "1k" H 6034 4080 50  0000 L CNN
-F 2 "" H 5975 4125 50  0001 C CNN
+F 2 "Resistor_SMD:R_0603_1608Metric_Pad0.98x0.95mm_HandSolder" H 5975 4125 50  0001 C CNN
 F 3 "~" H 5975 4125 50  0001 C CNN
 	1    5975 4125
@@
 $EndComp
 $Comp
-L Device:R_Small R?
+L Device:R_Small R24
 U 1 1 61A857F1
 P 5975 4375
-F 0 "R?" H 6034 4421 50  0000 L CNN
+F 0 "R24" H 6034 4421 50  0000 L CNN
 F 1 "620" H 6034 4330 50  0000 L CNN
-F 2 "" H 5975 4375 50  0001 C CNN
+F 2 "Resistor_SMD:R_0603_1608Metric_Pad0.98x0.95mm_HandSolder" H 5975 4375 50  0001 C CNN
 F 3 "~" H 5975 4375 50  0001 C CNN
 	1    5975 4375
@@
 +3.3V_ISO
 $Comp
-L eec:Transformer_1P_2S_WE_750313973 T?
+L eec:Transformer_1P_2S_WE_750313973 T1
 U 1 1 61AB5502
 P 5850 2400
-F 0 "T?" H 5850 2981 50  0000 C CNN
+F 0 "T1" H 5850 2981 50  0000 C CNN
 F 1 "Transformer_1P_2S_WE_750313973" H 5850 2890 50  0000 C CNN
-F 2 "" H 5850 2400 50  0001 C CNN
+F 2 "eec:750313973" H 5850 2400 50  0001 C CNN
 F 3 "~" H 5850 2400 50  0001 C CNN
 	1    5850 2400

Commit message: Footprints aangepast. Tekening aangepast
Parts:
- added C16: 100n, Capacitor_SMD:C_0603_1608Metric_Pad1.08x0.95mm_HandSolder, symbol Device:C_Small
- added C17: 1n, Capacitor_SMD:C_0603_1608Metric_Pad1.08x0.95mm_HandSolder, symbol Device:C_Small
- C10: footprint (none) -> Capacitor_THT:CP_Radial_D10.0mm_P5.00mm
- C11: footprint (none) -> Capacitor_SMD:C_1812_4532Metric_Pad1.57x3.40mm_HandSolder
- C12: footprint (none) -> Capacitor_SMD:C_1206_3216Metric_Pad1.33x1.80mm_HandSolder
Connections:
- net GNDS: now also C16.2, C17.2
- net +3.3V renamed +3V3
- net +3.3V_ISO renamed +3.3VP
- net +3.3VP: now also C16.1, C17.1
- net VCC renamed +VDC
- net VSS renamed GND1
Other:
- moved on the sheet: R21, R22, R25
